File: 3340_vco.kicad_pcb (KiCad board)
At the start: 2 copper layers, 40 x 98.8 mm, 68 parts, among them J1 Conn_01x10, J10 TRI OUT, J11 SAW OUT, J12 EXT PWM CONTROL IN, J2 SYNC IN, J5 FM IN, J6 1V/OCT IN, J7 CV2 IN, J9 SQ OUT, SW1 OCTAVES, SW2 SYNC_TYPE, U1 AS3340, U2 TL074

Commit message: BOM updated with correct resistor values
Parts:
- R11: value 1M5 -> 1M2
Changed lines of the file:
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@@
         (effects (font (size 1 1) (thickness 0.15)))
     )
-    (fp_text value "1M5" (at 1.27 2.37 90) (layer "F.Fab")
+    (fp_text value "1M2" (at 1.27 2.37 90) (layer "F.Fab")
         (effects (font (size 1 1) (thickness 0.15)))
     )
